Commit message: Att chefbot para pegasus, para poder compilar o original junto no msm ws

File: pegasus_description/urdf/pegasus_base.urdf.xacro (robot description, xacro)
@@ -6,8 +6,8 @@
       kobuki_description/launch/view_model.launch
  -->
-<robot name="chefbot" xmlns:xacro="http://ros.org/wiki/xacro">
-  <xacro:include filename="$(find chefbot_description)/urdf/common_properties.urdf.xacro"/>
-  <xacro:include filename="$(find chefbot_description)/urdf/chefbot_base_gazebo.urdf.xacro"/>
-  <!-- Chefbot -->
+<robot name="pegasus" xmlns:xacro="http://ros.org/wiki/xacro">
+  <xacro:include filename="$(find pegasus_description)/urdf/common_properties.urdf.xacro"/>
+  <xacro:include filename="$(find pegasus_description)/urdf/pegasus_base_gazebo.urdf.xacro"/>
+  <!-- pegasus -->
   <xacro:macro name="kobuki">
     <link name="base_footprint"/>
@@ -30,5 +30,5 @@
         <geometry>
           <!-- new mesh -->
-          <mesh filename="package://chefbot_description/meshes/base_plate.dae" />
+          <mesh filename="package://pegasus_description/meshes/base_plate.dae" />
         </geometry>
 <!--        <origin xyz="0.001 0 0.05199" rpy="0 0 ${M_PI/2}"/> -->
@@ -59,12 +59,12 @@
     <joint name="wheel_left_joint" type="continuous">
       <parent link="base_link"/>
-      <child link="chefbot_wheel_left_link"/>
+      <child link="pegasus_wheel_left_link"/>
       <origin xyz="0 ${0.28/2} 0.026" rpy="${-M_PI/2} 0 0"/>
       <axis xyz="0 0 1"/>
     </joint>
-    <link name="chefbot_wheel_left_link">
+    <link name="pegasus_wheel_left_link">
       <visual>
         <geometry>
-          <mesh filename="package://chefbot_description/meshes/wheel.dae"/>
+          <mesh filename="package://pegasus_description/meshes/wheel.dae"/>
         </geometry>
         <origin xyz="0 0 0" rpy="0 0 0"/>
@@ -86,12 +86,12 @@
     <joint name="wheel_right_joint" type="continuous">
       <parent link="base_link"/>
-      <child link="chefbot_wheel_right_link"/>
+      <child link="pegasus_wheel_right_link"/>
       <origin xyz="0.00 -${0.28/2} 0.026" rpy="${-M_PI/2} 0 0"/>
       <axis xyz="0 0 1"/>
     </joint>
-    <link name="chefbot_wheel_right_link">
+    <link name="pegasus_wheel_right_link">
       <visual>
         <geometry>
-          <mesh filename="package://chefbot_description/meshes/wheel.dae"/>
+          <mesh filename="package://pegasus_description/meshes/wheel.dae"/>
         </geometry>
         <origin xyz="0 0 0" rpy="0 0 0"/>
@@ -227,8 +227,8 @@
     <joint name="caster_front_joint" type="fixed">
       <parent link="base_link"/>
-      <child link="chefbot_caster_front_link"/>
+      <child link="pegasus_caster_front_link"/>
       <origin xyz="0.115 0.0 0.007" rpy="${-M_PI/2} 0 0"/>
     </joint>
-    <link name="chefbot_caster_front_link">
+    <link name="pegasus_caster_front_link">
       <collision>
         <geometry>
@@ -245,10 +245,10 @@
       </inertial>
     </link>
-    <joint name="chefbot_caster_back_joint" type="fixed">
-      <parent link="base_link"/>
-      <child link="chefbot_caster_back_link"/>
+    <joint name="pegasus_caster_back_joint" type="fixed">
+      <parent link="base_link"/>
+      <child link="pegasus_caster_back_link"/>
       <origin xyz="-0.135 0.0 0.009" rpy="${-M_PI/2} 0 0"/>
     </joint>
-    <link name="chefbot_caster_back_link">
+    <link name="pegasus_caster_back_link">
       <collision>
         <geometry>

File: pegasus_description/urdf/pegasus_base.xacro (robot description, xacro)
@@ -1,3 +1,3 @@
-<?xml version="1.0"?>
+<?xml version="1.0
 <!--
     - Base      : kobuki
@@ -7,5 +7,5 @@
 <robot name="turtlebot" xmlns:xacro="http://ros.org/wiki/xacro">
 <!--  <xacro:include filename="$(find turtlebot_description)/urdf/turtlebot_library.urdf.xacro" /> -->
-  <xacro:include filename="$(find chefbot_description)/urdf/chefbot_rviz_library.urdf.xacro" />
+  <xacro:include filename="$(find pegasus_description)/urdf/pegasus_rviz_library.urdf.xacro" />
   <!--kobuki/>
   <stack_hexagons parent="base_link"/>

File: pegasus_description/urdf/pegasus_base_gazebo.urdf.xacro (robot description, xacro)
@@ -2,5 +2,5 @@
 <robot name="kobuki_sim" xmlns:xacro="http://ros.org/wiki/xacro">
   <xacro:macro name="kobuki_sim">
-	  <gazebo reference="chefbot_wheel_left_link">
+	  <gazebo reference="pegasus_wheel_left_link">
 	    <mu1>1.0</mu1>
 	    <mu2>1.0</mu2>
@@ -10,5 +10,5 @@
 	    <maxVel>1.0</maxVel>
 	  </gazebo>
-	  <gazebo reference="chefbot_wheel_right_link">
+	  <gazebo reference="pegasus_wheel_right_link">
 	    <mu1>1.0</mu1>
 	    <mu2>1.0</mu2>
@@ -18,5 +18,5 @@
 	    <maxVel>1.0</maxVel>
 	  </gazebo>
-	  <gazebo reference="chefbot_caster_front_link">
+	  <gazebo reference="pegasus_caster_front_link">
 	    <mu1>0.0</mu1>
 	    <mu2>0.0</mu2>
@@ -26,5 +26,5 @@
 	    <maxVel>1.0</maxVel>
 	  </gazebo>
-	  <gazebo reference="chefbot_caster_back_link">
+	  <gazebo reference="pegasus_caster_back_link">
 	    <mu1>0.0</mu1>
 	    <mu2>0.0</mu2>

File: pegasus_description/urdf/pegasus_rviz_base.urdf.xacro (robot description, xacro)
@@ -1,5 +1,5 @@
 <?xml version='1.0'?>
-<robot name="chefbot" xmlns:xacro="http://www.ros.org/wiki/xacro">
-  <xacro:include filename="$(find chefbot_description)/urdf/common_properties.urdf.xacro" />
+<robot name="pegasus" xmlns:xacro="http://www.ros.org/wiki/xacro">
+  <xacro:include filename="$(find pegasus_description)/urdf/common_properties.urdf.xacro" />
 	<!-- Robot's part -->
 			<!-- Joint's -->
@@ -221,5 +221,5 @@
 		<origin xyz="0 0 0.075" rpy="0 0 0"/>
 			<geometry>
-				<mesh filename="package://chefbot_description/meshes/hokuyo.dae"/>
+				<mesh filename="package://pegasus_description/meshes/hokuyo.dae"/>
 			</geometry>
 		</visual>

Commit message: Merge New_urdf v1

File: pegasus_description/urdf/pegasus_base.urdf.xacro (robot description, xacro)
@@ -1,14 +1,8 @@
 <?xml version="1.0" ?>
-<!--
-  This is not a standalone urdf for kobuki. It simply defines the 'kobuki' tag that can
-  be incorporated by other urdf files (e.g. turtlebot).
-  See kobuki_standalone.urdf.xacro for a standalone urdf to be tested with
-      kobuki_description/launch/view_model.launch
- -->
 <robot name="pegasus" xmlns:xacro="http://ros.org/wiki/xacro">
   <xacro:include filename="$(find pegasus_description)/urdf/common_properties.urdf.xacro"/>
-  <xacro:include filename="$(find pegasus_description)/urdf/pegasus_base_gazebo.urdf.xacro"/>
+  <!--xacro:include filename="$(find pegasus_description)/urdf/pegasus_base_gazebo.urdf.xacro"/-->
   <!-- pegasus -->
-  <xacro:macro name="kobuki">
+  <!--xacro:macro name="kobuki"-->
     <link name="base_footprint"/>
     <!--
@@ -324,5 +318,5 @@
     </link>
     <!-- Kobuki Gazebo simulation details -->
-    <kobuki_sim/>
-  </xacro:macro>
+    <!--kobuki_sim/-->
+  <!--/xacro:macro-->
 </robot>
