Commit message: mudei o static TF no inicial e add no urdf o lidar, all tf lidar rviz NO

File: pegasus_description/urdf/mobot_w_lidar.xacro (robot description, xacro)
@@ -1,9 +1,273 @@
 <?xml version="1.0"?>
+<!-- <robot xmlns:xacro="http://www.ros.org/wiki/xacro" name="mobot"> <xacro:include filename="$(find pegasus_description)/urdf/mobot_xacro_defs.xacro"/> <xacro:include filename="$(find pegasus_description)/urdf/mobot_static_links.xacro"/>
+<xacro:include filename="$(find pegasus_description)/urdf/mobot_wheels.xacro"/> <xacro:include filename="$(find pegasus_description)/urdf/casters.xacro"/> -->
+<!--xacro:include filename="$(find mobot_urdf)/urdf/gazebo_tags.xacro" /-->
+<!--xacro:include filename="$(find pegasus_description)/urdf/add_lidar.xacro" /-->
+<!-- </robot> -->
 <robot xmlns:xacro="http://www.ros.org/wiki/xacro" name="mobot">
-  <xacro:include filename="$(find pegasus_description)/urdf/mobot_xacro_defs.xacro"/>
-  <xacro:include filename="$(find pegasus_description)/urdf/mobot_static_links.xacro"/>
-  <xacro:include filename="$(find pegasus_description)/urdf/mobot_wheels.xacro"/>
-  <xacro:include filename="$(find pegasus_description)/urdf/casters.xacro"/>
-  <!--xacro:include filename="$(find mobot_urdf)/urdf/gazebo_tags.xacro" /-->
-  <!--xacro:include filename="$(find pegasus_description)/urdf/add_lidar.xacro" /-->
+  <!-- define the base-link origin to lie at floor level, between the drive wheels-->
+  <!--main body is a simple box; origin is a center of box-->
+  <xacro:property name="bodylen" value="0.5461"/>
+  <xacro:property name="bodywidth" value="0.4572"/>
+  <xacro:property name="bodyheight" value="0.2"/>
+  <xacro:property name="bodyclearance" value="0.4"/>
+  <!--clearance from bottom of box to ground-->
+  <!-- derived values-->
+  <xacro:property name="half_bodylen" value="${bodylen/2.0}"/>
+  <xacro:property name="half_bodyheight" value="${bodyheight/2.0}"/>
+  <!-- placement of main body relative to base link frame -->
+  <xacro:property name="bodyOX" value="${-half_bodylen}"/>
+  <xacro:property name="bodyOY" value="0"/>
+  <xacro:property name="bodyOZ" value="0.45"/>
+  <!-- define the drive-wheel dimensions-->
+  <xacro:property name="tirediam" value="0.3302"/>
+  <xacro:property name="tirerad" value="${tirediam/2.0}"/>
+  <xacro:property name="tirewidth" value="0.06985"/>
+  <!-- "track" is the distance between the drive wheels -->
+  <xacro:property name="track" value=".56515"/>
+  <!-- battery box dimensions -->
+  <xacro:property name="batterylen" value="0.381"/>
+  <xacro:property name="batterywidth" value="0.3556"/>
+  <xacro:property name="batteryheight" value="0.254"/>
+  <!-- placement of battery box relative to base frame -->
+  <xacro:property name="batOX" value="-0.05"/>
+  <xacro:property name="batOY" value="0"/>
+  <xacro:property name="batOZ" value="0.22"/>
+  <xacro:property name="M_PI" value="3.1415926535897931"/>
+  <xacro:property name="boschwidth" value="0.0381"/>
+  <xacro:property name="casterdrop" value="0.125"/>
+  <xacro:property name="bracketwidth" value="0.1175"/>
+  <xacro:property name="bracketheight" value="0.16"/>
+  <xacro:property name="bracketthick" value="0.0508"/>
+  <xacro:property name="bracketangle" value="0.7854"/>
+  <xacro:property name="casterwidth" value="0.0826"/>
+  <xacro:property name="casterdiam" value="0.2286"/>
+  <!--here is a default inertia matrix with small, but legal values; use this when don't need accuracy for I -->
+  <!--model will assign inertia matrix dominated by main body box -->
+  <xacro:macro name="default_inertial" params="mass">
+    <inertial>
+      <mass value="${mass}"/>
+      <inertia ixx="0.01" ixy="0.0" ixz="0.0" iyy="0.01" iyz="0.0" izz="0.01"/>
+    </inertial>
+  </xacro:macro>
+  <xacro:macro name="wheel" params="prefix reflect">
+    <link name="${prefix}_wheel">
+      <visual>
+        <geometry>
+          <cylinder radius="${tirerad}" length="${tirewidth}"/>
+        </geometry>
+      </visual>
+      <collision>
+        <geometry>
+          <cylinder radius="${tirerad}" length="${tirewidth}"/>
+        </geometry>
+      </collision>
+      <inertial>
+        <!--assign inertial properties to drive wheels -->
+        <mass value="1"/>
+        <inertia ixx="0.1" ixy="0" ixz="0" iyy="0.1" iyz="0" izz="0.1"/>
+      </inertial>
+    </link>
+    <joint name="${prefix}_wheel_joint" type="continuous">
+      <axis xyz="0 0 1"/>
+      <parent link="base_link"/>
+      <child link="${prefix}_wheel"/>
+      <origin xyz="0 ${reflect*track/2} ${tirerad}" rpy="0 ${M_PI/2} ${M_PI/2}"/>
+      <limit effort="100" velocity="15"/>
+      <joint_properties damping="0.0" friction="0.0"/>
+    </joint>
+  </xacro:macro>
+  <xacro:macro name="caster" params="prefix reflect">
+    <link name="castdrop_${prefix}">
+      <visual>
+        <geometry>
+          <box size="${boschwidth} ${boschwidth} ${casterdrop}"/>
+        </geometry>
+        <origin xyz="0 0 0" rpy="0 0 0"/>
+      </visual>
+      <collision>
+        <geometry>
+          <box size="${boschwidth} ${boschwidth} ${casterdrop}"/>
+        </geometry>
+        <origin xyz="0 0 0" rpy="0 0 0"/>
+      </collision>
+      <xacro:default_inertial mass="0.2"/>
+    </link>
+    <joint name="cast2base_${prefix}" type="fixed">
+      <parent link="base_link"/>
+      <child link="castdrop_${prefix}"/>
+      <origin xyz="${-bodylen/2+bodyOX+boschwidth/2} ${reflect*bodywidth/2-reflect*boschwidth/2} ${-casterdrop/2-bodyheight/2+bodyOZ}"/>
+    </joint>
+    <link name="brackettop_${prefix}">
+      <visual>
+        <geometry>
+          <box size="${bracketwidth} ${bracketthick} .005"/>
+        </geometry>
+        <origin xyz="0 0 0" rpy="0 0 0"/>
+      </visual>
+      <collision>
+        <geometry>
+          <box size="${bracketwidth} ${bracketthick} .005"/>
+        </geometry>
+        <origin xyz="0 0 0" rpy="0 0 0"/>
+      </collision>
+      <xacro:default_inertial mass="0.2"/>
+    </link>
+    <joint name="cast2bracket_${prefix}" type="continuous">
+      <axis xyz="0 0 1"/>
+      <parent link="castdrop_${prefix}"/>
+      <child link="brackettop_${prefix}"/>
+      <origin xyz="0 0 ${-casterdrop/2}" rpy="0 0 ${M_PI/2}"/>
+      <joint_properties damping="0.0" friction="0.0"/>
+    </joint>
+    <link name="bracketside1_${prefix}">
+      <visual>
+        <geometry>
+          <box size="${bracketthick} ${bracketheight} .005"/>
+        </geometry>
+        <origin xyz="0 0 0" rpy="${M_PI/2} ${-bracketangle} ${M_PI/2}"/>
+      </visual>
+      <collision>
+        <geometry>
+          <box size="${bracketthick} ${bracketheight} .005"/>
+        </geometry>
+        <origin xyz="0 0 0" rpy="${M_PI/2} ${-bracketangle} ${M_PI/2}"/>
+      </collision>
+      <xacro:default_inertial mass="0.2"/>
+    </link>
+    <joint name="brack2top1_${prefix}" type="fixed">
+      <parent link="brackettop_${prefix}"/>
+      <child link="bracketside1_${prefix}"/>
+      <origin xyz="${bracketwidth/2} .04 -${bracketheight/2-.02}" rpy="0 0 0"/>
+    </joint>
+    <link name="bracketside2_${prefix}">
+      <visual>
+        <geometry>
+          <box size="${bracketthick} ${bracketheight} .005"/>
+        </geometry>
+        <origin xyz="0 0 0" rpy="${M_PI/2} ${-bracketangle} ${M_PI/2}"/>
+      </visual>
+      <collision>
+        <geometry>
+          <box size="${bracketthick} ${bracketheight} .005"/>
+        </geometry>
+        <origin xyz="0 0 0" rpy="${M_PI/2} ${-bracketangle} ${M_PI/2}"/>
+      </collision>
+      <xacro:default_inertial mass="0.2"/>
+    </link>
+    <joint name="brack2top2_${prefix}" type="fixed">
+      <parent link="brackettop_${prefix}"/>
+      <child link="bracketside2_${prefix}"/>
+      <origin xyz="${-bracketwidth/2} .04 -${bracketheight/2-.02}" rpy="0 0 0"/>
+    </joint>
+    <link name="${prefix}_casterwheel">
+      <visual>
+        <geometry>
+          <cylinder radius="${casterdiam/2}" length="${casterwidth}"/>
+        </geometry>
+      </visual>
+      <collision>
+        <geometry>
+          <cylinder radius="${casterdiam/2}" length="${casterwidth}"/>
+        </geometry>
+      </collision>
+      <!-- accept default inertial properties for caster wheels-->
+      <xacro:default_inertial mass="0.5"/>
+    </link>
+    <joint name="${prefix}_caster_joint" type="continuous">
+      <axis xyz="0 0 1"/>
+      <parent link="bracketside1_${prefix}"/>
+      <child link="${prefix}_casterwheel"/>
+      <origin xyz="${-casterwidth/2-.02} .053 -.053" rpy="0 ${M_PI/2} 0"/>
+      <limit effort="100" velocity="15"/>
+      <joint_properties damping="0.0" friction="0.0"/>
+    </joint>
+  </xacro:macro>
+  <xacro:caster prefix="left" reflect="1"/>
+  <xacro:caster prefix="right" reflect="-1"/>
+  <link name="base_link">
+    <visual>
+      <geometry>
+        <box size="${bodylen} ${bodywidth} ${bodyheight}"/>
+      </geometry>
+      <origin xyz="${bodyOX} ${bodyOY} ${bodyOZ}" rpy="0 0 0"/>
+    </visual>
+    <collision>
+      <geometry>
+        <box size="${bodylen} ${bodywidth} ${bodyheight}"/>
+      </geometry>
+      <origin xyz="${bodyOX} ${bodyOY} ${bodyOZ}" rpy="0 0 0"/>
+    </collision>
+    <inertial>
+      <!--assign almost all the mass to the main body box; set m= 100kg; treat I as approx m*r^2 -->
+      <mass value="100"/>
+      <inertia ixx="10" ixy="0" ixz="0" iyy="10" iyz="0" izz="10"/>
+    </inertial>
+  </link>
+  <xacro:wheel prefix="left" reflect="1"/>
+  <xacro:wheel prefix="right" reflect="-1"/>
+  <link name="batterybox">
+    <visual>
+      <geometry>
+        <box size="${batterylen} ${batterywidth} ${batteryheight}"/>
+      </geometry>
+      <origin xyz="0 0 0" rpy="0 0 0"/>
+    </visual>
+    <collision>
+      <geometry>
+        <box size="${batterylen} ${batterywidth} ${batteryheight}"/>
+      </geometry>
+      <origin xyz="0 0 0" rpy="0 0 0"/>
+    </collision>
+    <xacro:default_inertial mass="1"/>
+  </link>
+  <joint name="batterytobase" type="fixed">
+    <parent link="base_link"/>
+    <child link="batterybox"/>
+    <origin xyz="${batOX} ${batOY} ${batOZ}" rpy="0 0 0"/>
+  </joint>
+  <!-- <gazebo> <plugin name="differential_drive_controller" filename="libgazebo_ros_diff_drive.so"> <alwaysOn>true</alwaysOn> <updateRate>100</updateRate> <leftJoint>right_wheel_joint</leftJoint> <rightJoint>left_wheel_joint</rightJoint>
+  <wheelSeparation>${track}</wheelSeparation> <wheelDiameter>${tirediam}</wheelDiameter> <torque>200</torque> <commandTopic>cmd_vel</commandTopic> <odometryTopic>odom</odometryTopic> <odometryFrame>odom</odometryFrame>
+  <robotBaseFrame>base_link</robotBaseFrame> -->
+  <!--don't publish wheel TF, so it does not conflict with robot_state_publisher -->
+  <!-- <publishWheelTF>false</publishWheelTF> <publishWheelJointState>true</publishWheelJointState> </plugin> </gazebo> -->
+  <!-- <gazebo reference="right_wheel"> <mu1>100000.0</mu1> <mu2>100000.0</mu2> <material>Gazebo/Black</material> </gazebo> <gazebo reference="left_wheel"> <mu1>100000.0</mu1> <mu2>100000.0</mu2> <material>Gazebo/Black</material> </gazebo> <gazebo
+  reference="right_casterwheel"> <mu1>100000.0</mu1> <mu2>100000.0</mu2> <material>Gazebo/Black</material> </gazebo> <gazebo reference="left_casterwheel"> <mu1>100000.0</mu1> <mu2>100000.0</mu2> <material>Gazebo/Black</material> </gazebo> <gazebo>
+  <plugin name="joint_state_publisher" filename="libgazebo_ros_joint_state_publisher.so"> <jointName>cast2bracket_right, cast2bracket_left, right_caster_joint, left_caster_joint </jointName> </plugin> </gazebo> -->
+  <!-- add a simulated lidar, including visual, collision and inertial properties, and physics simulation-->
+  <link name="lidar_link">
+    <collision>
+      <origin xyz="0 0 0" rpy="0 0 0"/>
+      <geometry>
+        <!-- coarse LIDAR model; a simple box -->
+        <box size="0.2 0.2 0.2"/>
+      </geometry>
+    </collision>
+    <visual>
+      <origin xyz="0 0 0" rpy="0 0 0"/>
+      <geometry>
+        <box size="0.2 0.2 0.2"/>
+      </geometry>
+      <material name="sick_grey">
+        <color rgba="0.7 0.5 0.3 1.0"/>
+      </material>
+    </visual>
+    <inertial>
+      <mass value="4.0"/>
+      <origin xyz="0 0 0" rpy="0 0 0"/>
+      <inertia ixx="0.01" ixy="0" ixz="0" iyy="0.01" iyz="0" izz="0.01"/>
+    </inertial>
+  </link>
+  <!--the above displays a box meant to imply Lidar-->
+  <joint name="lidar_joint" type="fixed">
+    <axis xyz="0 1 0"/>
+    <origin xyz="0.1 0 0.56" rpy="0 0 0"/>
+    <parent link="base_link"/>
+    <child link="lidar_link"/>
+  </joint>
+  <!-- here is the gazebo plug-in to simulate a lidar sensor -->
+  <!-- <gazebo reference="lidar_link"> <sensor type="gpu_ray" name="sick_lidar_sensor"> <pose>0 0 0 0 0 0</pose> <visualize>false</visualize> <update_rate>40</update_rate> <ray> <scan> <horizontal> <samples>181</samples> <resolution>1</resolution>
+  <min_angle>-1.570796</min_angle> <max_angle>1.570796</max_angle> </horizontal> </scan> <range> <min>0.10</min> <max>80.0</max> <resolution>0.01</resolution> </range> <noise> <type>gaussian</type> <mean>0.0</mean> <stddev>0.01</stddev> </noise> </ray>
+  -->
+  <!-- <plugin name="gazebo_ros_lidar_controller" filename="libgazebo_ros_gpu_laser.so"> <topicName>/scan</topicName> <frameName>lidar_link</frameName> </plugin> </sensor> </gazebo> -->
 </robot>
