Commit message: Chefbot urdf with my config at other things

File: pegasus_description/robots/chefbot_circles_kinect.urdf.xacro (robot description, xacro)
@@ -6,6 +6,5 @@
 -->
 <robot name="turtlebot" xmlns:xacro="http://ros.org/wiki/xacro">
-<!--  <xacro:include filename="$(find turtlebot_description)/urdf/turtlebot_library.urdf.xacro" /> -->
-  <xacro:include filename="$(find pegasus_description)/urdf/pegasus_rviz_library.urdf.xacro" />
+  <xacro:include filename="$(find chefbot_description)/urdf/chefbot_library.urdf.xacro" />
   <kobuki/>
   <stack_hexagons parent="base_link"/>

File: pegasus_description/urdf/pegasus_base.urdf.xacro (robot description, xacro)
@@ -1,8 +1,14 @@
 <?xml version="1.0" ?>
+<!--
+  This is not a standalone urdf for kobuki. It simply defines the 'kobuki' tag that can
+  be incorporated by other urdf files (e.g. turtlebot).
+  See kobuki_standalone.urdf.xacro for a standalone urdf to be tested with
+      kobuki_description/launch/view_model.launch
+ -->
 <robot name="pegasus" xmlns:xacro="http://ros.org/wiki/xacro">
   <xacro:include filename="$(find pegasus_description)/urdf/common_properties.urdf.xacro"/>
-  <!--xacro:include filename="$(find pegasus_description)/urdf/pegasus_base_gazebo.urdf.xacro"/-->
+  <xacro:include filename="$(find pegasus_description)/urdf/pegasus_base_gazebo.urdf.xacro"/>
   <!-- pegasus -->
-  <!--xacro:macro name="kobuki"-->
+  <xacro:macro name="kobuki">
     <link name="base_footprint"/>
     <!--
@@ -318,5 +324,5 @@
     </link>
     <!-- Kobuki Gazebo simulation details -->
-    <!--kobuki_sim/-->
-  <!--/xacro:macro-->
+    <kobuki_sim/>
+  </xacro:macro>
 </robot>

File: pegasus_description/urdf/pegasus_rviz_base.urdf.xacro (robot description, xacro)
@@ -1,232 +1,328 @@
-<?xml version='1.0'?>
-<robot name="pegasus" xmlns:xacro="http://www.ros.org/wiki/xacro">
-  <xacro:include filename="$(find pegasus_description)/urdf/common_properties.urdf.xacro" />
-	<!-- Robot's part -->
-			<!-- Joint's -->
-	  		<!-- Base footprint -->
-	<joint name="base_joint" type="fixed">
-		<origin xyz="0 0 0.0102" rpy="0 0 0" />
-		<parent link="base_footprint"/>
-		<child link="base_link" />
-	</joint>
-		  	<!-- Caster wheels -->
-		  	<!-- Left wheels -->
-	<joint name="left_axle_joint" type="fixed">
-		<origin xyz="0 0.171475 0.0178" rpy="0 0 0"/>
-		<parent link="base_link"/>
-		<child link="left_axle_link"/>
-		<axis xyz="0 1 0"/>
-	</joint>
-	<joint name="left_wheel_joint" type="fixed">
-		<origin xyz="0 0.01905 0" rpy="0 0 0"/>
-		<parent link="left_axle_link"/>
-		<child link="left_wheel_link"/>
-		<axis xyz="0 1 0"/>
-	</joint>
-		  	<!-- Right wheels -->
-	<joint name="right_axle_joint" type="fixed">
-		<origin xyz="0 -0.171475 0.0178" rpy="0 0 0"/>
-		<parent link="base_link"/>
-		<child link="right_axle_link"/>
-		<axis xyz="0 1 0"/>
-	</joint>
-	<joint name="right_wheel_joint" type="fixed">
-		<origin xyz="0 -0.01905 0" rpy="0 0 0"/>
-		<parent link="right_axle_link"/>
-		<child link="right_wheel_link"/>
-		<axis xyz="0 1 0"/>
-	</joint>
-		<!--Sensors -->
-	<joint name="laser_joint" type="fixed">
-		<axis xyz="0 1 0" />
-		<origin xyz=".15 0 .1" rpy="0 0 0"/>
-		<parent link="base_link"/>
-		<child link="laser_link"/>
-	</joint>
-		<!-- Link's -->
-  		<!-- Base footprint -->
-	<link name="base_footprint"/>
-     		<!-- Chassis -->
-	<link name='base_link'>
-		<pose>0 0 0.1 0 0 0</pose>
-		<inertial>
-		<mass value="15.0"/>
-		<origin xyz="0.0 0 0.1" rpy=" 0 0 0"/>
-		<inertia
-		  ixx="0.1" ixy="0" ixz="0"
-		  iyy="0.1" iyz="0"
-		  izz="0.1"
-		/>
-		</inertial>
-		<collision>
-		<geometry>
-		<box size=".96 .665 .08"/>
-		</geometry>
-		</collision>
-		<visual>
-		<origin xyz="0 0 0" rpy=" 0 0 0"/>
-		<geometry>
-		<box size=".96 .665 .08"/>
-		</geometry>
-		</visual>
-		  	<!-- Caster wheels -->
-		<collision name='caster_collision'>
-		<origin xyz="-0.3 -0.25 0" rpy=" 0 0 0"/>
-			<geometry>
-				<sphere radius="0.065"/>
-			</geometry>
-			<surface>
-			<friction>
-				<ode>
-					<mu>0</mu>
-					<mu2>0</mu2>
-					<slip1>1.0</slip1>
-					<slip2>1.0</slip2>
-				</ode>
-			</friction>
-			</surface>
-		</collision>
-		<visual name='caster_visual'>
-		<origin xyz="-0.3 -0.25 0" rpy=" 0 0 0"/>
-			<geometry>
-				<sphere radius="0.065"/>
-			</geometry>
-		</visual>
-		<collision name='caster_front_collision'>
-		<origin xyz="-0.3 0.25 0" rpy=" 0 0 0"/>
-			<geometry>
-				<sphere radius="0.065"/>
-			</geometry>
-			<surface>
-			<friction>
-				<ode>
-					<mu>0</mu>
-					<mu2>0</mu2>
-					<slip1>1.0</slip1>
-					<slip2>1.0</slip2>
-				</ode>
-			</friction>
-			</surface>
-		</collision>
-		<visual name='caster_front_visual'>
-		<origin xyz="-0.3 0.25 0" rpy=" 0 0 0"/>
-			<geometry>
-				<sphere radius="0.065"/>
-			</geometry>
-		</visual>
-	</link>
-	  	<!-- Left wheels -->
-	<link name="left_axle_link">
-		<inertial>
-      		<origin xyz="0 0 0" rpy="0 1.5707 1.5707"/>
-			<mass value="5" />
-			<inertia
-				ixx=".1" ixy="0.0" ixz="0.0"
-				iyy=".1" iyz="0.0"
-				izz=".1"/>
-		</inertial>
-		<visual>
-      		<origin xyz="0.38 0.104 0" rpy="0 1.5707 1.5707"/>
-			<geometry>
-				<cylinder radius="0.077" length="0.05"/>
-			</geometry>
-			<material name ="light_grey" />
-		</visual>
-		<collision>
-      		<origin xyz="0.38 0.104 0" rpy="0 1.5707 1.5707"/>
-			<geometry>
-				<cylinder radius="0.077" length="0.05"/>
-			</geometry>
-		</collision>
-	</link>
-	<link name="left_wheel_link">
-		<inertial>
-		<origin xyz="0 0 0" rpy="0 1.5707 1.5707"/>
-			<mass value="5" />
-			<inertia
-			ixx=".1" ixy="0.0" ixz="0.0"
-			iyy=".1" iyz="0.0"
-			izz=".1"/>
-		</inertial>
-		<visual>
-		<origin xyz="0.38 0.104 0" rpy="0 1.5707 1.5707"/>
-			<geometry>
-				<cylinder radius="0.077" length="0.05"/>
-			</geometry>
-			<material name ="black" />
-		</visual>
-		<collision>
-		<origin xyz="0.38 0.104 0" rpy="0 1.5707 1.5707"/>
-			<geometry>
-				<cylinder radius="0.077" length="0.05"/>
-			</geometry>
-		</collision>
-	</link>
-	  	<!-- Right wheels -->
-	<link name="right_axle_link">
-		<inertial>
-      		<origin xyz="0 0 0" rpy="0 1.5707 1.5707"/>
-			<mass value="5" />
-			<inertia
-				ixx=".1" ixy="0.0" ixz="0.0"
-				iyy=".1" iyz="0.0"
-				izz=".1"/>
-		</inertial>
-		<visual>
-      		<origin xyz="0.38 -0.104 0" rpy="0 1.5707 1.5707"/>
-			<geometry>
-				<cylinder radius="0.077" length="0.05"/>
-			</geometry>
-			<material name ="light_grey" />
-		</visual>
-		<collision>
-      		<origin xyz="0.38 -0.104 0" rpy="0 1.5707 1.5707"/>
-			<geometry>
-				<cylinder radius="0.077" length="0.05"/>
-			</geometry>
-		</collision>
-	</link>
-	<link name="right_wheel_link">
-		<inertial>
-      		<origin xyz="0 0 0" rpy="0 1.5707 1.5707"/>
-			<mass value="5" />
-			<inertia
-				ixx=".1" ixy="0.0" ixz="0.0"
-				iyy=".1" iyz="0.0"
-				izz=".1"/>
-		</inertial>
-		<visual>
-      		<origin xyz="0.38 -0.104 0" rpy="0 1.5707 1.5707"/>
-			<geometry>
-				<cylinder radius="0.077" length="0.05"/>
-			</geometry>
-			<material name ="black" />
-		</visual>
-		<collision>
-      		<origin xyz="0.38 -0.104 0" rpy="0 1.5707 1.5707"/>
-			<geometry>
-				<cylinder radius="0.077" length="0.05"/>
-			</geometry>
-		</collision>
-	</link>
-		<!-- Hokuyo Laser -->
-	<link name="laser_link">
-		<collision>
-			<origin xyz="0 0 0" rpy="0 0 0"/>
-			<geometry>
-				<box size="0.1 0.1 0.1"/>
-			</geometry>
-		</collision>
-		<visual>
-		<origin xyz="0 0 0.075" rpy="0 0 0"/>
-			<geometry>
-				<mesh filename="package://pegasus_description/meshes/hokuyo.dae"/>
-			</geometry>
-		</visual>
-	<inertial>
-	<mass value="1e-5" />
-	<origin xyz="0 0 0" rpy="0 0 0"/>
-	<inertia ixx="1e-6" ixy="0" ixz="0" iyy="1e-6" iyz="0" izz="1e-6" />
-	</inertial>
-	</link>
+<?xml version="1.0" ?>
+<!--
+  This is not a standalone urdf for kobuki. It simply defines the 'kobuki' tag that can
+  be incorporated by other urdf files (e.g. turtlebot).
+  See kobuki_standalone.urdf.xacro for a standalone urdf to be tested with
+      kobuki_description/launch/view_model.launch
+ -->
+<robot name="pegasus" xmlns:xacro="http://ros.org/wiki/xacro">
+  <xacro:include filename="$(find pegasus_description)/urdf/common_properties.urdf.xacro"/>
+  <xacro:include filename="$(find pegasus_description)/urdf/pegasus_base_gazebo.urdf.xacro"/>
+  <!-- pegasus -->
+  <xacro:macro name="kobuki">
+    <link name="base_footprint"/>
+    <!--
+       Base link is set at the bottom of the base mould.
+       This is done to be compatible with the way base link
+       was configured for turtlebot 1. Refer to
+       https://github.com/turtlebot/turtlebot/issues/40
+       To put the base link at the more oft used wheel
+       axis, set the z-distance from the base_footprint
+       to 0.352.
+      -->
+    <joint name="base_joint" type="fixed">
+      <origin xyz="0 0 0.0102" rpy="0 0 0" />
+      <parent link="base_footprint"/>
+      <child link="base_link" />
+    </joint>
+    <link name="base_link">
+      <visual>
+        <geometry>
+          <!-- new mesh -->
+          <mesh filename="package://pegasus_description/meshes/base_plate.dae" />
+        </geometry>
+<!--        <origin xyz="0.001 0 0.05199" rpy="0 0 ${M_PI/2}"/> -->
+	 <origin xyz="0.001 0 -0.034" rpy="0 0 ${M_PI/2}"/>
+      </visual>
+      <collision>
+        <geometry>
+          <cylinder length="0.10938" radius="0.178"/>
+        </geometry>
+        <origin xyz="0.0 0 0.05949" rpy="0 0 0"/>
+      </collision>
+      <inertial>
+        <!-- COM experimentally determined -->
+        <origin xyz="0.01 0 0"/>
+        <mass value="2.4"/> <!-- 2.4/2.6 kg for small/big battery pack -->
+        <!-- Kobuki's inertia tensor is approximated by a cylinder with homogeneous mass distribution
+             More details: http://en.wikipedia.org/wiki/List_of_moment_of_inertia_tensors
+             m = 2.4 kg; h = 0.09 m; r = 0.175 m
+             ixx = 1/12 * m * (3 * r^2 + h^2)
+             iyy = 1/12 * m * (3 * r^2 + h^2)
+             izz = 1/2 * m * r^2
+          -->
+        <inertia ixx="0.019995" ixy="0.0" ixz="0.0"
+                 iyy="0.019995" iyz="0.0"
+                 izz="0.03675" />
+      </inertial>
+    </link>
+<!--
+    <joint name="wheel_left_joint" type="continuous">
+      <parent link="base_link"/>
+      <child link="pegasus_wheel_left_link"/>
+      <origin xyz="0 ${0.28/2} 0.026" rpy="${-M_PI/2} 0 0"/>
+      <axis xyz="0 0 1"/>
+    </joint>
+    <link name="pegasus_wheel_left_link">
+      <visual>
+        <geometry>
+          <mesh filename="package://pegasus_description/meshes/wheel.dae"/>
+        </geometry>
+        <origin xyz="0 0 0" rpy="0 0 0"/>
+      </visual>
+      <collision>
+        <geometry>
+          <cylinder length="0.0206" radius="0.0352"/>
+        </geometry>
+        <origin rpy="0 0 0" xyz="0 0 0"/>
+      </collision>
+      <inertial>
+        <mass value="0.01" />
+        <origin xyz="0 0 0" />
+        <inertia ixx="0.001" ixy="0.0" ixz="0.0"
+                 iyy="0.001" iyz="0.0"
+                 izz="0.001" />
+      </inertial>
+    </link>
+    <joint name="wheel_right_joint" type="continuous">
+      <parent link="base_link"/>
+      <child link="pegasus_wheel_right_link"/>
+      <origin xyz="0.00 -${0.28/2} 0.026" rpy="${-M_PI/2} 0 0"/>
+      <axis xyz="0 0 1"/>
+    </joint>
+    <link name="pegasus_wheel_right_link">
+      <visual>
+        <geometry>
+          <mesh filename="package://pegasus_description/meshes/wheel.dae"/>
+        </geometry>
+        <origin xyz="0 0 0" rpy="0 0 0"/>
+      </visual>
+      <collision>
+        <geometry>
+          <cylinder length="0.0206" radius="0.0350"/>
+        </geometry>
+        <origin rpy="0 0 0" xyz="0 0 0"/>
+      </collision>
+      <inertial>
+        <mass value="0.01" />
+        <origin xyz="0 0 0" />
+        <inertia ixx="0.001" ixy="0.0" ixz="0.0"
+                 iyy="0.001" iyz="0.0"
+                 izz="0.001" />
+      </inertial>
+    </link>
+-->
+	  <link name="left_axle_link">
+	    <inertial>
+	      <origin xyz="0 -0.035 0.021"/>
+	      <mass value="0.01" />
+	      <inertia ixx="0.001" ixy="0.0" ixz="0.0"
+	        iyy="0.001" iyz="0.0" izz="0.001" />
+	    </inertial>
+	    <visual>
+	      <origin xyz="0 -0.035 0.021" rpy="0 1.5707 1.5707" />
+	      <geometry>
+            <cylinder radius="0.0045" length = "0.02"/>
+	      </geometry>
+          <material name ="light_grey" />
+	    </visual>
+	    <collision>
+	      <origin xyz="0 -0.035 0.021" rpy="0 1.5707 1.5707" />
+	      <geometry>
+            <cylinder radius="0.00635" length = "0.00635"/>
+	      </geometry>
+	    </collision>
+	  </link>
+	  <joint name="left_axle_joint" type="fixed">
+	    <origin xyz="0 0.171475 0.0178" rpy="0 0 0"/>
+	    <parent link="base_link"/>
+	    <child link="left_axle_link"/>
+	    <axis xyz="0 1 0"/>
+	  </joint>
+	  <link name="right_axle_link">
+	    <inertial>
+	      <origin xyz="0 0.035 0.021"/>
+	      <mass value="0.01" />
+	      <inertia ixx="0.001" ixy="0.0" ixz="0.0"
+	        iyy="0.001" iyz="0.0" izz="0.001" />
+	    </inertial>
+	    <visual>
+	      <origin xyz="0 0.035 0.02" rpy="0 1.5707 1.5707" />
+	      <geometry>
+            <cylinder radius="0.0045" length = "0.002"/>
+	      </geometry>
+          <material name ="light_grey" />
+	    </visual>
+	    <collision>
+	      <origin xyz="0 0.035 0.02" rpy="0 1.5707 1.5707" />
+	      <geometry>
+            <cylinder radius="0.0045" length = "0.002"/>
+	      </geometry>
+	    </collision>
+	  </link>
+	  <joint name="right_axle_joint" type="fixed">
+	    <origin xyz="0 -0.171475 0.0178" rpy="0 0 0"/>
+	    <parent link="base_link"/>
+	    <child link="right_axle_link"/>
+	    <axis xyz="0 1 0"/>
+	  </joint>
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
File: pegasus_description/urdf/pegasus_rviz_library.urdf.xacro (robot description, xacro)
@@ -6,6 +6,17 @@
   <!-- General -->
   <xacro:include filename="$(find pegasus_description)/urdf/common_properties.urdf.xacro"/>
-  <!--xacro:include filename="$(find pegasus_description)/urdf/pegasus_properties.urdf.xacro"/-->
+  <xacro:include filename="$(find pegasus_description)/urdf/pegasus_properties.urdf.xacro"/>
+<!-- Need changes in pegasus base and circle -->
   <!-- Bases -->
   <xacro:include filename="$(find pegasus_description)/urdf/pegasus_rviz_base.urdf.xacro"/>
+<!--  <xacro:include filename="$(find create_description)/urdf/create.urdf.xacro"/>
+  <xacro:include filename="$(find kobuki_description)/urdf/kobuki.urdf.xacro" />
+-->
+  <!-- Stacks -->
+<!--  <xacro:include filename="$(find pegasus_description)/urdf/circles.urdf.xacro"/>  -->
+<!-- <xacro:include filename="$(find pegasus_description)/urdf/stacks/circles.urdf.xacro"/> -->
+<!--  <xacro:include filename="$(find turtlebot_description)/urdf/stacks/hexagons.urdf.xacro"/> -->
+  <!-- 3D Sensors -->
+  <xacro:include filename="$(find pegasus_description)/urdf/sensors/kinect.urdf.xacro"/>
+  <xacro:include filename="$(find pegasus_description)/urdf/sensors/asus_xtion_pro.urdf.xacro"/>
 </robot>
