Commit message: possuem o chefbot original e a adaptação tb

File: chefbot/chefbot_description/urdf/bkup/chefbot_base.urdf.xacro (robot description, xacro)
@@ -6,9 +6,9 @@
       kobuki_description/launch/view_model.launch
  -->
-<robot name="pegasus" xmlns:xacro="http://ros.org/wiki/xacro">
-  <xacro:include filename="$(find pegasus_description)/urdf/common_properties.urdf.xacro"/>
-  <xacro:include filename="$(find pegasus_description)/urdf/pegasus_base_gazebo.urdf.xacro"/>
-  <!-- pegasus -->
-  <!--xacro:macro name="kobuki"-->
+<robot name="kobuki" xmlns:xacro="http://ros.org/wiki/xacro">
+  <xacro:include filename="$(find chefbot_description)/urdf/common_properties.urdf.xacro"/>
+  <xacro:include filename="$(find chefbot_description)/urdf/chefbot_base_gazebo.urdf.xacro"/>
+  <!-- Kobuki -->
+  <xacro:macro name="kobuki">
     <link name="base_footprint"/>
     <!--
@@ -30,5 +30,5 @@
         <geometry>
           <!-- new mesh -->
-          <mesh filename="package://pegasus_description/meshes/base_plate.dae" />
+          <mesh filename="package://chefbot_description/meshes/base_plate.dae" />
         </geometry>
 <!--        <origin xyz="0.001 0 0.05199" rpy="0 0 ${M_PI/2}"/> -->
@@ -59,12 +59,12 @@
     <joint name="wheel_left_joint" type="continuous">
       <parent link="base_link"/>
-      <child link="pegasus_wheel_left_link"/>
+      <child link="wheel_left_link"/>
       <origin xyz="0 ${0.28/2} 0.026" rpy="${-M_PI/2} 0 0"/>
       <axis xyz="0 0 1"/>
     </joint>
-    <link name="pegasus_wheel_left_link">
+    <link name="wheel_left_link">
       <visual>
         <geometry>
-          <mesh filename="package://pegasus_description/meshes/wheel.dae"/>
+          <mesh filename="package://chefbot_description/meshes/wheel.dae"/>
         </geometry>
         <origin xyz="0 0 0" rpy="0 0 0"/>
@@ -86,12 +86,12 @@
     <joint name="wheel_right_joint" type="continuous">
       <parent link="base_link"/>
-      <child link="pegasus_wheel_right_link"/>
+      <child link="wheel_right_link"/>
       <origin xyz="0.00 -${0.28/2} 0.026" rpy="${-M_PI/2} 0 0"/>
       <axis xyz="0 0 1"/>
     </joint>
-    <link name="pegasus_wheel_right_link">
+    <link name="wheel_right_link">
       <visual>
         <geometry>
-          <mesh filename="package://pegasus_description/meshes/wheel.dae"/>
+          <mesh filename="package://chefbot_description/meshes/wheel.dae"/>
         </geometry>
         <origin xyz="0 0 0" rpy="0 0 0"/>
@@ -111,124 +111,10 @@
       </inertial>
     </link>
-<!--
-	  <link name="left_axle_link">
-	    <inertial>
-	      <origin xyz="0 0 0"/>
-	      <mass value="0.01" />
-	      <inertia ixx="0.001" ixy="0.0" ixz="0.0"
-	        iyy="0.001" iyz="0.0" izz="0.001" />
-	    </inertial>
-	    <visual>
-	      <origin xyz="0 0 0" rpy="0 1.5707 1.5707" />
-	      <geometry>
-            <cylinder radius="0.00635" length = "0.00635"/>
-	      </geometry>
-          <material name ="light_grey" />
-	    </visual>
-	    <collision>
-	      <origin xyz="0 0 0" rpy="0 1.5707 1.5707" />
-	      <geometry>
-            <cylinder radius="0.00635" length = "0.00635"/>
-	      </geometry>
-	    </collision>
-	  </link>
-	  <joint name="left_axle_joint" type="fixed">
-	    <origin xyz="0 0.171475 0.0178" rpy="0 0 0"/>
-	    <parent link="base_link"/>
-	    <child link="left_axle_link"/>
-	    <axis xyz="0 1 0"/>
-	  </joint>
-	  <link name="right_axle_link">
-	    <inertial>
-	      <origin xyz="0 0 0"/>
-	      <mass value="0.01" />
-	      <inertia ixx="0.001" ixy="0.0" ixz="0.0"
-	        iyy="0.001" iyz="0.0" izz="0.001" />
-	    </inertial>
-	    <visual>
-	      <origin xyz="0 0 0" rpy="0 1.5707 1.5707" />
-	      <geometry>
-            <cylinder radius="0.00635" length = "0.00635"/>
-	      </geometry>
-          <material name ="light_grey" />
-	    </visual>
-	    <collision>
-	      <origin xyz="0 0 0" rpy="0 1.5707 1.5707" />
-	      <geometry>
-            <cylinder radius="0.00635" length = "0.00635"/>
-	      </geometry>
-	    </collision>
-	  </link>
-	  <joint name="right_axle_joint" type="fixed">
-	    <origin xyz="0 -0.171475 0.0178" rpy="0 0 0"/>
-	    <parent link="base_link"/>
-	    <child link="right_axle_link"/>
-	    <axis xyz="0 1 0"/>
-	  </joint>
-	  <link name="left_wheel_link">
-	    <inertial>
-	      <origin xyz="0 0 0"/>
-	      <mass value="0.01" />
-	      <inertia ixx="0.001" ixy="0.0" ixz="0.0"
-	        iyy="0.001" iyz="0.0" izz="0.001" />
-	    </inertial>
-	    <visual>
-	      <origin xyz="0 0 0" rpy="0 1.5707 1.5707" />
-	      <geometry>
-            <cylinder radius="0.0762" length = "0.03175"/>
-	      </geometry>
-          <material name ="black" />
-	    </visual>
-	    <collision>
-	      <origin xyz="0 0 0" rpy="0 1.5707 1.5707" />
-	      <geometry>
-            <cylinder radius="0.0762" length = "0.03175"/>
-	      </geometry>
-	    </collision>
-	  </link>
-        -->
-<!--	  <joint name="left_wheel_joint" type="fixed">
-	    <origin xyz="0 0.01905 0" rpy="0 0 0"/>
-	    <parent link="left_axle_link"/>
-	    <child link="left_wheel_link"/>
-	    <axis xyz="0 1 0"/>
-	  </joint>
-	  <link name="right_wheel_link">
-	    <inertial>
-	      <origin xyz="0 0 0"/>
-	      <mass value="0.01" />
-	      <inertia ixx="0.001" ixy="0.0" ixz="0.0"
-	        iyy="0.001" iyz="0.0" izz="0.001" />
-	    </inertial>
-	    <visual>
-	      <origin xyz="0 0 0" rpy="0 1.5707 1.5707" />
-	      <geometry>
-            <cylinder radius="0.0762" length = "0.03175"/>
-	      </geometry>
-          <material name ="black" />
-	    </visual>
-	    <collision>
-	      <origin xyz="0 0 0" rpy="0 1.5707 1.5707" />
-	      <geometry>
-            <cylinder radius="0.0762" length = "0.03175"/>
-	      </geometry>
-	    </collision>
-	  </link>
-	-->
-        <!-- Fixed because we never rotate it anyway, it is just for show -->
-        <!-- NOTE This may prevent gazebo from working with this model -->
-<!--	  <joint name="right_wheel_joint" type="fixed">
-	    <origin xyz="0 -0.01905 0" rpy="0 0 0"/>
-	    <parent link="right_axle_link"/>
-	    <child link="right_wheel_link"/>
-	    <axis xyz="0 1 0"/>
-	  </joint>
--->
     <joint name="caster_front_joint" type="fixed">
       <parent link="base_link"/>
-      <child link="pegasus_caster_front_link"/>
+      <child link="caster_front_link"/>
       <origin xyz="0.115 0.0 0.007" rpy="${-M_PI/2} 0 0"/>
     </joint>
-    <link name="pegasus_caster_front_link">
+    <link name="caster_front_link">
       <collision>
         <geometry>
@@ -245,10 +131,10 @@
       </inertial>
     </link>
-    <joint name="pegasus_caster_back_joint" type="fixed">
-      <parent link="base_link"/>
-      <child link="pegasus_caster_back_link"/>
+    <joint name="caster_back_joint" type="fixed">
+      <parent link="base_link"/>
+      <child link="caster_back_link"/>
       <origin xyz="-0.135 0.0 0.009" rpy="${-M_PI/2} 0 0"/>
     </joint>
-    <link name="pegasus_caster_back_link">
+    <link name="caster_back_link">
       <collision>
         <geometry>
@@ -325,4 +211,4 @@
     <!-- Kobuki Gazebo simulation details -->
     <kobuki_sim/>
-  <!--/xacro:macro-->
+  </xacro:macro>
 </robot>

File: chefbot/chefbot_description/urdf/chefbot_base.urdf.xacro (robot description, xacro)
@@ -6,9 +6,9 @@
       kobuki_description/launch/view_model.launch
  -->
-<robot name="pegasus" xmlns:xacro="http://ros.org/wiki/xacro">
-  <xacro:include filename="$(find pegasus_description)/urdf/common_properties.urdf.xacro"/>
-  <xacro:include filename="$(find pegasus_description)/urdf/pegasus_base_gazebo.urdf.xacro"/>
-  <!-- pegasus -->
-  <!--xacro:macro name="kobuki"-->
+<robot name="chefbot" xmlns:xacro="http://ros.org/wiki/xacro">
+  <xacro:include filename="$(find chefbot_description)/urdf/common_properties.urdf.xacro"/>
+  <xacro:include filename="$(find chefbot_description)/urdf/chefbot_base_gazebo.urdf.xacro"/>
+  <!-- Chefbot -->
+  <xacro:macro name="kobuki">
     <link name="base_footprint"/>
     <!--
@@ -30,5 +30,5 @@
         <geometry>
           <!-- new mesh -->
-          <mesh filename="package://pegasus_description/meshes/base_plate.dae" />
+          <mesh filename="package://chefbot_description/meshes/base_plate.dae" />
         </geometry>
 <!--        <origin xyz="0.001 0 0.05199" rpy="0 0 ${M_PI/2}"/> -->
@@ -59,12 +59,12 @@
     <joint name="wheel_left_joint" type="continuous">
       <parent link="base_link"/>
-      <child link="pegasus_wheel_left_link"/>
+      <child link="chefbot_wheel_left_link"/>
       <origin xyz="0 ${0.28/2} 0.026" rpy="${-M_PI/2} 0 0"/>
       <axis xyz="0 0 1"/>
     </joint>
-    <link name="pegasus_wheel_left_link">
+    <link name="chefbot_wheel_left_link">
       <visual>
         <geometry>
-          <mesh filename="package://pegasus_description/meshes/wheel.dae"/>
+          <mesh filename="package://chefbot_description/meshes/wheel.dae"/>
         </geometry>
         <origin xyz="0 0 0" rpy="0 0 0"/>
@@ -86,12 +86,12 @@
     <joint name="wheel_right_joint" type="continuous">
       <parent link="base_link"/>
-      <child link="pegasus_wheel_right_link"/>
+      <child link="chefbot_wheel_right_link"/>
       <origin xyz="0.00 -${0.28/2} 0.026" rpy="${-M_PI/2} 0 0"/>
       <axis xyz="0 0 1"/>
     </joint>
-    <link name="pegasus_wheel_right_link">
+    <link name="chefbot_wheel_right_link">
       <visual>
         <geometry>
-          <mesh filename="package://pegasus_description/meshes/wheel.dae"/>
+          <mesh filename="package://chefbot_description/meshes/wheel.dae"/>
         </geometry>
         <origin xyz="0 0 0" rpy="0 0 0"/>
@@ -227,8 +227,8 @@
     <joint name="caster_front_joint" type="fixed">
       <parent link="base_link"/>
-      <child link="pegasus_caster_front_link"/>
+      <child link="chefbot_caster_front_link"/>
       <origin xyz="0.115 0.0 0.007" rpy="${-M_PI/2} 0 0"/>
     </joint>
-    <link name="pegasus_caster_front_link">
+    <link name="chefbot_caster_front_link">
       <collision>
         <geometry>
@@ -245,10 +245,10 @@
       </inertial>
     </link>
-    <joint name="pegasus_caster_back_joint" type="fixed">
-      <parent link="base_link"/>
-      <child link="pegasus_caster_back_link"/>
+    <joint name="chefbot_caster_back_joint" type="fixed">
+      <parent link="base_link"/>
+      <child link="chefbot_caster_back_link"/>
       <origin xyz="-0.135 0.0 0.009" rpy="${-M_PI/2} 0 0"/>
     </joint>
-    <link name="pegasus_caster_back_link">
+    <link name="chefbot_caster_back_link">
       <collision>
         <geometry>
@@ -325,4 +325,4 @@
     <!-- Kobuki Gazebo simulation details -->
     <kobuki_sim/>
-  <!--/xacro:macro-->
+  </xacro:macro>
 </robot>

File: chefbot/chefbot_description/urdf/chefbot_rviz_base.urdf.xacro (robot description, xacro)
@@ -6,9 +6,9 @@
       kobuki_description/launch/view_model.launch
  -->
-<robot name="pegasus" xmlns:xacro="http://ros.org/wiki/xacro">
-  <xacro:include filename="$(find pegasus_description)/urdf/common_properties.urdf.xacro"/>
-  <xacro:include filename="$(find pegasus_description)/urdf/pegasus_base_gazebo.urdf.xacro"/>
-  <!-- pegasus -->
-  <!--xacro:macro name="kobuki"-->
+<robot name="chefbot" xmlns:xacro="http://ros.org/wiki/xacro">
+  <xacro:include filename="$(find chefbot_description)/urdf/common_properties.urdf.xacro"/>
+  <xacro:include filename="$(find chefbot_description)/urdf/chefbot_base_gazebo.urdf.xacro"/>
+  <!-- Chefbot -->
+  <xacro:macro name="kobuki">
     <link name="base_footprint"/>
     <!--
@@ -30,5 +30,5 @@
         <geometry>
           <!-- new mesh -->
-          <mesh filename="package://pegasus_description/meshes/base_plate.dae" />
+          <mesh filename="package://chefbot_description/meshes/base_plate.dae" />
         </geometry>
 <!--        <origin xyz="0.001 0 0.05199" rpy="0 0 ${M_PI/2}"/> -->
@@ -57,14 +57,15 @@
       </inertial>
     </link>
+<!--
     <joint name="wheel_left_joint" type="continuous">
       <parent link="base_link"/>
-      <child link="pegasus_wheel_left_link"/>
+      <child link="chefbot_wheel_left_link"/>
       <origin xyz="0 ${0.28/2} 0.026" rpy="${-M_PI/2} 0 0"/>
       <axis xyz="0 0 1"/>
     </joint>
-    <link name="pegasus_wheel_left_link">
+    <link name="chefbot_wheel_left_link">
       <visual>
         <geometry>
-          <mesh filename="package://pegasus_description/meshes/wheel.dae"/>
+          <mesh filename="package://chefbot_description/meshes/wheel.dae"/>
         </geometry>
         <origin xyz="0 0 0" rpy="0 0 0"/>
@@ -86,12 +87,12 @@
     <joint name="wheel_right_joint" type="continuous">
       <parent link="base_link"/>
-      <child link="pegasus_wheel_right_link"/>
+      <child link="chefbot_wheel_right_link"/>
       <origin xyz="0.00 -${0.28/2} 0.026" rpy="${-M_PI/2} 0 0"/>
       <axis xyz="0 0 1"/>
     </joint>
-    <link name="pegasus_wheel_right_link">
+    <link name="chefbot_wheel_right_link">
       <visual>
         <geometry>
-          <mesh filename="package://pegasus_description/meshes/wheel.dae"/>
+          <mesh filename="package://chefbot_description/meshes/wheel.dae"/>
         </geometry>
         <origin xyz="0 0 0" rpy="0 0 0"/>
@@ -111,8 +112,8 @@
       </inertial>
     </link>
-<!--
+-->
 	  <link name="left_axle_link">
 	    <inertial>
-	      <origin xyz="0 0 0"/>
+	      <origin xyz="0 -0.035 0.021"/>
 	      <mass value="0.01" />
 	      <inertia ixx="0.001" ixy="0.0" ixz="0.0"
@@ -120,12 +121,12 @@
 	    </inertial>
 	    <visual>
-	      <origin xyz="0 0 0" rpy="0 1.5707 1.5707" />
-	      <geometry>
-            <cylinder radius="0.00635" length = "0.00635"/>
+	      <origin xyz="0 -0.035 0.021" rpy="0 1.5707 1.5707" />
+	      <geometry>
+            <cylinder radius="0.0045" length = "0.02"/>
 	      </geometry>
           <material name ="light_grey" />
 	    </visual>
 	    <collision>
-	      <origin xyz="0 0 0" rpy="0 1.5707 1.5707" />
+	      <origin xyz="0 -0.035 0.021" rpy="0 1.5707 1.5707" />
 	      <geometry>
             <cylinder radius="0.00635" length = "0.00635"/>
@@ -141,5 +142,5 @@
 	  <link name="right_axle_link">
 	    <inertial>
-	      <origin xyz="0 0 0"/>
+	      <origin xyz="0 0.035 0.021"/>
 	      <mass value="0.01" />
 	      <inertia ixx="0.001" ixy="0.0" ixz="0.0"
@@ -147,14 +148,14 @@
 	    </inertial>
 	    <visual>
-	      <origin xyz="0 0 0" rpy="0 1.5707 1.5707" />
-	      <geometry>
-            <cylinder radius="0.00635" length = "0.00635"/>
+	      <origin xyz="0 0.035 0.02" rpy="0 1.5707 1.5707" />
+	      <geometry>
+            <cylinder radius="0.0045" length = "0.002"/>
 	      </geometry>
           <material name ="light_grey" />
 	    </visual>
 	    <collision>
-	      <origin xyz="0 0 0" rpy="0 1.5707 1.5707" />
-	      <geometry>
-            <cylinder radius="0.00635" length = "0.00635"/>
+	      <origin xyz="0 0.035 0.02" rpy="0 1.5707 1.5707" />
+	      <geometry>
+            <cylinder radius="0.0045" length = "0.002"/>
 	      </geometry>
 	    </collision>
@@ -168,5 +169,5 @@
 	  <link name="left_wheel_link">
 	    <inertial>
-	      <origin xyz="0 0 0"/>
+	      <origin xyz="0 -0.035 0.021"/>
 	      <mass value="0.01" />
 	      <inertia ixx="0.001" ixy="0.0" ixz="0.0"
@@ -174,12 +175,12 @@
 	    </inertial>
 	    <visual>
-	      <origin xyz="0 0 0" rpy="0 1.5707 1.5707" />
-	      <geometry>
-            <cylinder radius="0.0762" length = "0.03175"/>
+	      <origin xyz="0 -0.035 0.021" rpy="0 1.5707 1.5707" />
+	      <geometry>
+            <cylinder radius="0.045" length = "0.02"/>
 	      </geometry>
           <material name ="black" />
 	    </visual>
 	    <collision>
-	      <origin xyz="0 0 0" rpy="0 1.5707 1.5707" />
+	      <origin xyz="0 -0.035 0.021" rpy="0 1.5707 1.5707" />
 	      <geometry>
             <cylinder radius="0.0762" length = "0.03175"/>
@@ -187,6 +188,7 @@
 	    </collision>
 	  </link>
-        -->
-<!--	  <joint name="left_wheel_joint" type="fixed">
+        <!-- Fixed because we never rotate it anyway, it is just for show -->
+        <!-- NOTE This may prevent gazebo from working with this model -->
+	  <joint name="left_wheel_joint" type="fixed">
 	    <origin xyz="0 0.01905 0" rpy="0 0 0"/>
 	    <parent link="left_axle_link"/>
@@ -196,5 +198,5 @@
 	  <link name="right_wheel_link">
 	    <inertial>
-	      <origin xyz="0 0 0"/>
+	      <origin xyz="0 0.035 0.021"/>
 	      <mass value="0.01" />
 	      <inertia ixx="0.001" ixy="0.0" ixz="0.0"
@@ -202,21 +204,20 @@
 	    </inertial>
 	    <visual>
-	      <origin xyz="0 0 0" rpy="0 1.5707 1.5707" />
-	      <geometry>
-            <cylinder radius="0.0762" length = "0.03175"/>
+	      <origin xyz="0 0.035 0.021" rpy="0 1.5707 1.5707" />
+	      <geometry>
+            <cylinder radius="0.045" length = "0.02"/>
 	      </geometry>
           <material name ="black" />
 	    </visual>
 	    <collision>
-	      <origin xyz="0 0 0" rpy="0 1.5707 1.5707" />
-	      <geometry>
-            <cylinder radius="0.0762" length = "0.03175"/>
+	      <origin xyz="0 0.035 0.021" rpy="0 1.5707 1.5707" />
+	      <geometry>
+            <cylinder radius="0.045" length = "0.02"/>
 	      </geometry>
 	    </collision>
 	  </link>
-	-->
         <!-- Fixed because we never rotate it anyway, it is just for show -->
         <!-- NOTE This may prevent gazebo from working with this model -->
-<!--	  <joint name="right_wheel_joint" type="fixed">
+	  <joint name="right_wheel_joint" type="fixed">
 	    <origin xyz="0 -0.01905 0" rpy="0 0 0"/>
 	    <parent link="right_axle_link"/>
@@ -224,11 +225,10 @@
 	    <axis xyz="0 1 0"/>
 	  </joint>
--->
     <joint name="caster_front_joint" type="fixed">
       <parent link="base_link"/>
-      <child link="pegasus_caster_front_link"/>
+      <child link="chefbot_caster_front_link"/>
       <origin xyz="0.115 0.0 0.007" rpy="${-M_PI/2} 0 0"/>
     </joint>
-    <link name="pegasus_caster_front_link">
+    <link name="chefbot_caster_front_link">
       <collision>
         <geometry>
@@ -245,10 +245,10 @@
       </inertial>
     </link>
-    <joint name="pegasus_caster_back_joint" type="fixed">
-      <parent link="base_link"/>
-      <child link="pegasus_caster_back_link"/>
+    <joint name="chefbot_caster_back_joint" type="fixed">
+      <parent link="base_link"/>
+      <child link="chefbot_caster_back_link"/>
       <origin xyz="-0.135 0.0 0.009" rpy="${-M_PI/2} 0 0"/>
     </joint>
-    <link name="pegasus_caster_back_link">
+    <link name="chefbot_caster_back_link">
       <collision>
         <geometry>
@@ -325,4 +325,4 @@
     <!-- Kobuki Gazebo simulation details -->
     <kobuki_sim/>
-  <!--/xacro:macro-->
+  </xacro:macro>
 </robot>
